File: main/led_yol/led_yol.sch (KiCad schematic (older format))
At the start: 129 parts, among them J1 Power_Terminal, Q1 BS250, Q2 2N7000, Q3 2N7000, Q4 2N7000, Q5 2N7000, Q6 2N7000, Q7 2N7000, Q8 2N7000, Q9 2N7000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

Commit message: sebelum sampai ke percetakan
Parts:
- added J10, J7, J8, J9: GND_VIA, Connector_PinHeader_2.54mm:PinHeader_1x02_P2.54mm_Vertical, symbol Connector:Conn_01x02_Male
- added J2: VCC_VIA, Connector_PinHeader_2.54mm:PinHeader_1x02_P2.54mm_Vertical, symbol Connector:Conn_01x02_Male
- added J3: L_VIA, Connector_PinHeader_2.54mm:PinHeader_1x02_P2.54mm_Vertical, symbol Connector:Conn_01x02_Male
- added J4: A_VIA, Connector_PinHeader_2.54mm:PinHeader_1x02_P2.54mm_Vertical, symbol Connector:Conn_01x02_Male
- added J5: D_VIA, Connector_PinHeader_2.54mm:PinHeader_1x02_P2.54mm_Vertical, symbol Connector:Conn_01x02_Male
- added J6: N._VIA, Connector_PinHeader_2.54mm:PinHeader_1x02_P2.54mm_Vertical, symbol Connector:Conn_01x02_Male
- Q1, Q2, Q3, Q4, Q5, Q6, Q7, Q8, Q9: footprint Package_TO_SOT_THT:TO-92_Inline -> Package_TO_SOT_THT:TO-92_Inline_Wide
Connections:
- net +5V: now also J2.1 (Pin_1); no longer JP1.1, U3.20 (VCC)
- net GND: now also J10.2 (Pin_2), J7.2 (Pin_2), J8.2 (Pin_2); no longer D1.1 (K), JP1.3, Q2.1 (S), Q7.1 (S), U3.10 (GND)
- net O_A: now also J4.2 (Pin_2); no longer U3.8 (D3)
- net O_D: now also J5.2 (Pin_2); no longer U3.14 (D5)
- net O_L: now also J3.2 (Pin_2); no longer U3.7 (D2)
- net O_N.: now also J6.2 (Pin_2); no longer U3.17 (D6)
- new net 1_3GND: J9.1 (Pin_1), Q2.1 (S)
- new net 2_3GND: J10.1 (Pin_1), J9.2 (Pin_2), JP1.3
- new net 5V_VIA: J2.2 (Pin_2), JP1.1, U3.20 (VCC)
- new net GND1: D1.1 (K), J7.1 (Pin_1), U3.10 (GND)
- new net GND2: J8.1 (Pin_1), Q7.1 (S)
- new net O_VIA_A: J4.1 (Pin_1), U3.8 (D3)
- new net O_VIA_D: J5.1 (Pin_1), U3.14 (D5)
- new net O_VIA_L: J3.1 (Pin_1), U3.7 (D2)
- new net O_VIA_N.: J6.1 (Pin_1), U3.17 (D6)
