File: main/led_yol/led_yol.kicad_pcb (KiCad board)
At the start: 2 copper layers, 129 parts, among them J1 Power_Terminal, Q1 BS250, Q2 2N7000, Q3 2N7000, Q4 2N7000, Q5 2N7000, Q6 2N7000, Q7 2N7000, Q8 2N7000, Q9 2N7000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

Commit message: sebelum sampai ke percetakan
Parts:
- added J10: GND_VIA, Connector_PinHeader_2.54mm:PinHeader_1x02_P2.54mm_Vertical, F.Cu at (113.9, 164.2)
- added J2: VCC_VIA, Connector_PinHeader_2.54mm:PinHeader_1x02_P2.54mm_Vertical, F.Cu at (71.1, 154.7)
- added J3: L_VIA, Connector_PinHeader_2.54mm:PinHeader_1x02_P2.54mm_Vertical, F.Cu at (149.4, 173.3)
- added J4: A_VIA, Connector_PinHeader_2.54mm:PinHeader_1x02_P2.54mm_Vertical, F.Cu at (158.1, 173.3)
- added J5: D_VIA, Connector_PinHeader_2.54mm:PinHeader_1x02_P2.54mm_Vertical, F.Cu at (157.8, 156.0)
- added J6: N._VIA, Connector_PinHeader_2.54mm:PinHeader_1x02_P2.54mm_Vertical, F.Cu at (148.9, 156.0)
- added J7: GND_VIA, Connector_PinHeader_2.54mm:PinHeader_1x02_P2.54mm_Vertical, F.Cu at (179.7, 163.2)
- added J8: GND_VIA, Connector_PinHeader_2.54mm:PinHeader_1x02_P2.54mm_Vertical, F.Cu at (163.4, 150.6)
- added J9: GND_VIA, Connector_PinHeader_2.54mm:PinHeader_1x02_P2.54mm_Vertical, F.Cu at (96.2, 172.5)
- Q1, Q2, Q3, Q4, Q5, Q6, Q7, Q8, Q9: footprint Package_TO_SOT_THT:TO-92_Inline -> Package_TO_SOT_THT:TO-92_Inline_Wide
- moved D1 114.7 mm to (184.7, 169.0), turned to 270 degrees
- moved C4 60.1 mm to (197.2, 165.0)
- moved R1 60.1 mm to (211.1, 157.0)
- moved R2 60.1 mm to (190.3, 170.1)
- moved R3 60.1 mm to (226.0, 166.7)
- moved RV1 60.1 mm to (220.7, 168.4)
- moved U2 60.1 mm to (205.3, 162.4)
- moved D84 15.7 mm to (275.6, 122.6)
- moved D91 9.90 mm to (282.6, 129.6)
- moved JP1 7.80 mm to (132.3, 162.9)
- moved D92 7.00 mm to (289.6, 129.6)
- moved D93 7.00 mm to (289.6, 136.6)
- moved D94 7.00 mm to (289.6, 143.6)
- moved D95 7.00 mm to (296.6, 143.6)
- moved D75 6.00 mm to (241.6, 122.6)
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Connections:
- D1 pad 1: GND -> /GND1
- JP1 pad 1: +5V -> /5V_VIA
- JP1 pad 3: GND -> /2_3GND
- Q2 pad 1: GND -> /1_3GND
- Q7 pad 1: GND -> /GND2
- U3 pad 10: GND -> /GND1
- U3 pad 14: /O_D -> /O_VIA_D
- U3 pad 17: /O_N. -> /O_VIA_N.
- U3 pad 20: +5V -> /5V_VIA
- U3 pad 7: /O_L -> /O_VIA_L
- U3 pad 8: /O_A -> /O_VIA_A
Routing:
- net +24V: track 0.00 -> 406.9 mm
- net /INV_IN: track 205.5 -> 110.3 mm
- net +5V: track 147.5 -> 229.3 mm
- net /5V_VIA: track 0.00 -> 75.4 mm
- net /O_N.: track 169.9 -> 127.4 mm
- net /2_3GND: track 0.00 -> 41.0 mm
- net /CLOCK: track 85.2 -> 46.8 mm
- net Net-(D56-Pad1): track 0.00 -> 34.9 mm
- net Net-(D4-Pad1): track 0.00 -> 27.9 mm
- net Net-(D58-Pad1): track 74.0 -> 46.4 mm
- net /GND1: track 0.00 -> 26.6 mm
- net Net-(D64-Pad1): track 0.00 -> 20.1 mm
- net Net-(D35-Pad2): track 0.00 -> 18.8 mm
- net Net-(C4-Pad1): track 49.5 -> 68.2 mm
- net /1_3GND: track 0.00 -> 17.3 mm
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- added copper zone on B.Cu, net GND
Other:
- board outline added: 306.1 x 85.9 mm
- net class power added: clearance 0.254, trace_width 0.254, via_dia 0.8, via_drill 0.4

Commit message: Change track width
Parts:
- moved Q1 6.00 mm to (66.9, 163.9)
- moved Q2 6.00 mm to (79.6, 163.2)
Routing:
- net +5V: track 229.3 -> 236.5 mm
- net Net-(C4-Pad1): track 68.2 -> 74.8 mm
- net /1_3GND: track 17.3 -> 21.9 mm
- net /INV_IN: track 110.3 -> 112.5 mm
- net /CLOCK: track 46.8 -> 45.6 mm
- net Net-(R1-Pad2): track 17.9 -> 17.0 mm
- net Net-(D84-Pad1): track 15.8 -> 16.7 mm
- net Net-(D43-Pad2): track 14.3 -> 13.6 mm
Other:
- net class Default: trace_width 0.254 -> 0.3302; via_drill 0.4 -> 0.65
- net class power: trace_width 0.254 -> 0.3302; via_drill 0.4 -> 0.65
- rule pad_to_mask_clearance: 0.051 -> 0.254
- rule solder_mask_min_width: 0.25 -> 0.5
- rule trace_min: 0.254 -> 0.3302
- rule via_min_drill: 0.3 -> 0.65
- rule via_min_size: 0.4 -> 0.65
