File: main/led_agn/led_agn.kicad_pcb (KiCad board)
At the start: 2 copper layers, 164 parts, among them J1 Barrel_Jack_Switch, J2 Power_Terminal, Q1 BS250, Q2 2N7000, Q3 2N7000, Q4 2N7000, Q5 2N7000, Q6 2N7000, Q7 2N7000, Q8 2N7000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

Commit message: add already-placed design (before routing)
Parts:
- removed D119, D91: LED, LED_THT:LED_D3.0mm
- R24: value 100R -> 680R
- moved D1 212.5 mm to (269.1, 75.3), turned to 90 degrees
- moved R22 212.1 mm to (256.2, 26.7), turned to 225 degrees
- moved R24 208.3 mm to (263.5, 26.7), turned to 225 degrees
- moved R2 207.4 mm to (212.1, 99.9), turned to 45 degrees
- moved RV1 204.8 mm to (191.9, 98.8), turned to 180 degrees
- moved R3 200.3 mm to (204.6, 99.9), turned to 45 degrees
- moved R1 193.8 mm to (204.0, 92.7), turned to 225 degrees
- moved U2 184.1 mm to (132.1, 100.8), turned to 90 degrees
- moved R23 183.0 mm to (241.1, 33.9), turned to 45 degrees
- moved R21 177.4 mm to (229.7, 26.7), turned to 225 degrees
- moved R20 168.4 mm to (207.6, 33.9), turned to 45 degrees
- moved Q9 167.6 mm to (201.6, 84.1), turned to 90 degrees
- moved U1 165.4 mm to (176.6, 92.5)
- moved R19 165.1 mm to (222.4, 26.7), turned to 225 degrees
- moved C4 158.8 mm to (74.7, 100.6), turned to 180 degrees
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Connections:
- D118 pad 1: Net-(D118-Pad1) -> Net-(D107-Pad1)
- D92 pad 2: Net-(D91-Pad1) -> Net-(D92-Pad2)
- R20 pad 1: Net-(D91-Pad2) -> Net-(D92-Pad2)
Other:
- board outline added: 250.3 x 81.9 mm
- net class power added: clearance 0.254, trace_width 0.381, via_dia 0.8, via_drill 0.6

Commit message: after autoroute (before adding logo)
Parts:
- added REF**: 1Pin, Connector_Pin:Pin_D1.3mm_L11.0mm, F.Cu at (250.5, 100.4)
- added REF**: 1Pin, Connector_Pin:Pin_D1.3mm_L11.0mm, F.Cu at (46.0, 100.2)
- added REF**: 1Pin, Connector_Pin:Pin_D1.3mm_L11.0mm, F.Cu at (269.5, 28.6)
- added REF**: 1Pin, Connector_Pin:Pin_D1.3mm_L11.0mm, F.Cu at (26.8, 28.6)
Routing:
- net +12V: track 0.00 -> 348.8 mm
- net +5V: track 0.00 -> 224.0 mm
- net Net-(D107-Pad1): track 0.00 -> 82.8 mm
- net /INV_IN: track 0.00 -> 80.6 mm
- net Net-(D13-Pad1): track 0.00 -> 78.7 mm
- net /O_A: track 0.00 -> 78.7 mm
- net /O_H.: track 0.00 -> 72.0 mm
- net Net-(D101-Pad1): track 0.00 -> 68.5 mm
- net /CLOCK: track 0.00 -> 62.1 mm
- net Net-(D1-Pad2): track 0.00 -> 58.1 mm
- net /O_G: track 0.00 -> 51.3 mm
- net /O_K.: track 0.00 -> 42.8 mm
- net Net-(D25-Pad1): track 0.00 -> 41.5 mm
- net Net-(D42-Pad1): track 0.00 -> 39.4 mm
- net /O_S: track 0.00 -> 37.1 mm
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- added copper zone on B.Cu, net GND
Other:
- board size 250.3 x 81.9 mm -> 251.6 x 86.9 mm
- net class led added: clearance 0.254, trace_width 0.508, via_dia 0.8, via_drill 0.6
- net class power: trace_width 0.381 -> 0.762
- net class signal added: clearance 0.254, trace_width 0.381, via_dia 0.8, via_drill 0.6
- board text added: "A G N E S K R I S T I N A H A L O H O"
- board text added: "GND"
- board text added: "VCC"

Commit message: adding watermark, gerber file
Parts:
- added G***: LOGO, lib:cat_icon, F.Cu at (236.6, 90.6)
- added G***: KiCad Logo, lib:KiCad-Logo_11mmx5mm, F.Cu at (67.7, 21.7)
Other:
- board text added: "29/09/2019"
- board text added: "By :"
- board text added: "M E O W B O Y"
- board text added: "Running LED (version: 2.0)"
